File: Hardware/LegoLight_HQ/LegoLight_HQ.kicad_sch (KiCad schematic)
At the start: 5 parts, among them J1 Conn_02x15_Counter_Clockwise, SW1 SW_Push, SW2 SW_Push

Commit message: update pcbs
Parts:
- added C1: 10uf, Capacitor_SMD:C_0805_2012Metric, symbol Device:C
- added C2: 0.1uf, Capacitor_SMD:C_0805_2012Metric, symbol Device:C
- added J2, J3: I2C, SnapEDA Library:SPARKFUN_PRT-14417, symbol Connector_Generic:Conn_01x04
- added J4: VEML7700-TT, SnapEDA Library:XDCR_VEML7700-TT, symbol Connector_Generic:Conn_01x04
- J1: Mouser Part Number (none) -> M50-3001545
- R1, R2: Mouser Part Number (none) -> CR1206-FX-4701ELF
Connections:
- net +3.3V: now also C1.1, C2.1, J4.2 (Pin_2)
- net GND: now also C1.2, C2.2, J2.1 (Pin_1), J3.1 (Pin_1), J4.3 (Pin_3)
- net SCL: now also J2.4 (Pin_4), J3.4 (Pin_4), J4.1 (Pin_1)
- net SDA: now also J2.3 (Pin_3), J3.3 (Pin_3), J4.4 (Pin_4)
- net VBUS: now also J2.2 (Pin_2), J3.2 (Pin_2)
- net +BATT renamed BAT
