File: Hardware/LegoLight_HQ/LegoLight_HQ.kicad_pcb (KiCad board)
At the start: 2 copper layers, 64.1 x 56 mm, 5 parts, among them J1 Conn_02x15_Counter_Clockwise, SW1 SW_Push, SW2 SW_Push

Commit message: update pcbs
Parts:
- added C1: 10uf, Capacitor_SMD:C_0805_2012Metric, F.Cu at (45.6, 63.5)
- added C2: 0.1uf, Capacitor_SMD:C_0805_2012Metric, F.Cu at (48.6, 63.5)
- added J2: I2C, SnapEDA Library:SPARKFUN_PRT-14417, F.Cu at (32.8, 64.0)
- added J3: I2C, SnapEDA Library:SPARKFUN_PRT-14417, F.Cu at (91.3, 64.0)
- added J4: VEML7700-TT, SnapEDA Library:XDCR_VEML7700-TT, F.Cu at (81.5, 56.0)
- added REF1: MountingHole_3.2mm_M3_DIN965_Pad, MountingHole:MountingHole_3.2mm_M3_DIN965_Pad, F.Cu at (90.2, 54.0)
- added REF2: MountingHole_3.2mm_M3_DIN965_Pad, MountingHole:MountingHole_3.2mm_M3_DIN965_Pad, F.Cu at (34.0, 54.0)
- added REF3: MountingHole_3.2mm_M3_DIN965_Pad, MountingHole:MountingHole_3.2mm_M3_DIN965_Pad, F.Cu at (34.0, 102.0)
- turned R2 to 90 degrees
Connections:
- net +BATT renamed /BAT
Routing:
- net VBUS: track 0.00 -> 69.7 mm
- net /IO02: track 0.00 -> 65.3 mm
- net /SCL: track 0.00 -> 62.9 mm, vias 0 -> 1
- net /SDA: track 0.00 -> 62.6 mm, vias 0 -> 1
- net /IO01: track 0.00 -> 57.7 mm
- net +3.3V: track 0.00 -> 51.7 mm, vias 0 -> 1
- net /BAT: track 0.00 -> 1.27 mm
- net GND: vias 0 -> 23
- added copper zone on B.Cu, net GND
- added copper zone on F.Cu, net GND
Other:
- board text added: "0"
- board text added: "0.1uf"
- board text added: "10uf"
- board text added: "4.7k"
- board text added: "LegoLight HQ"
- board text added: "by Averrin"
- board text added: "rev"

Commit message: final?
Other:
- board text removed: "0"
- board text removed: "rev"
