File: Hardware/LegoLight_R3/ext_i2c.kicad_sch (KiCad schematic)
At the start: 9 parts, among them J10 I2C, J2 I2C, U5 PCA9306D

Commit message: update pcbs
Parts:
- J10, J2: footprint SnapEDA Library:ADAFRUIT_4328 -> SnapEDA Library:SPARKFUN_PRT-14417
- U5: Mouser Part Number 771-PCA9306DP-T -> 771-PCA9306DP-T
Changed lines of the file:
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@@
 			)
 		)
-		(property "Mouser Part Number" " 771-PCA9306DP-T"
+		(property "Mouser Part Number" "771-PCA9306DP-T"
 			(at 58.42 74.93 0)
 			(effects
@@
 			)
 		)
-		(property "Footprint" "SnapEDA Library:ADAFRUIT_4328"
+		(property "Footprint" "SnapEDA Library:SPARKFUN_PRT-14417"
 			(at 91.44 90.17 0)
 			(effects
@@
 			)
 		)
-		(property "Footprint" "SnapEDA Library:ADAFRUIT_4328"
+		(property "Footprint" "SnapEDA Library:SPARKFUN_PRT-14417"
 			(at 91.44 71.12 0)
 			(effects
