File: Hardware/LegoLight_R3/LegoLight_R3.kicad_pcb (KiCad board)
At the start: 2 copper layers, 30 x 65 mm, 83 parts, among them J1 USB4105-GF-A, J10 I2C, J11 Conn_01x02_Socket, J12 Conn_01x02_Socket, J13 Conn_01x02_Socket, J14 Conn_01x02_Socket, J15 Conn_01x02_Socket, J16 Conn_01x02_Socket, J17 Conn_01x02_Socket, J18 Conn_01x02_Socket, J19 Conn_01x02_Socket, J2 I2C, J20 Conn_01x02_Socket, J21 Conn_01x02_Socket, J22 Conn_01x02_Socket, J23 Conn_01x02_Socket, J24 Conn_01x02_Socket, J25 Conn_01x02_Socket, J26 Conn_01x02_Socket, J3 I2C, J4 SWD, J7 LED_EXT, U1 24LC01BT-I_OT, U2 PCA9685PW, U3 ATSAMD21E18A-A, U5 PCA9306D, Y1 32.768 kHz

Commit message: update pcbs
Parts:
- removed BTN2, BTN3: BTN, SnapEDA Library:SW_TL3305AF160QG
- removed D1: SK6812, LED_SMD:LED_SK6812_PLCC4_5.0x5.0mm_P3.2mm
- removed R11, R12: 10KOHM, Resistor_SMD:R_0805_2012Metric_Pad1.20x1.40mm_HandSolder
- removed RESET: TL3305AF160QG, SnapEDA Library:SW_TL3305AF160QG
- added C7: 3pf, Capacitor_SMD:C_0805_2012Metric, F.Cu at (197.6, 106.6)
- added C8: 3pf, Capacitor_SMD:C_0805_2012Metric, F.Cu at (196.6, 103.9)
- added J8: 103R012BB100, mouser:103R012BB100, B.Cu at (190.0, 90.0)
- added RESET1: TL3305AF160QG, mouser:B3U-1000P, F.Cu at (181.2, 94.6)
- added Y2: 32.768 kHz, Crystal:Crystal_SMD_MicroCrystal_CC8V-T1A-2Pin_2.0x1.2mm, F.Cu at (194.9, 106.9)
- BTN1: footprint SnapEDA Library:SW_TL3305AF160QG -> mouser:B3U-1000P
- J10, J2, J7: footprint SnapEDA Library:ADAFRUIT_4328 -> SnapEDA Library:SPARKFUN_PRT-14417
- J3: value I2C -> 103R012BB100; footprint SnapEDA Library:ADAFRUIT_4328 -> mouser:103R012BB100; moved to B.Cu
- JP2: moved to F.Cu
- R16, R3: footprint Resistor_SMD:R_0805_2012Metric_Pad1.20x1.40mm_HandSolder -> Resistor_SMD:R_0402_1005Metric_Pad0.72x0.64mm_HandSolder
- U1: footprint Package_TO_SOT_SMD:SOT-353_SC-70-5_Handsoldering -> Package_TO_SOT_SMD:SOT-353_SC-70-5
- moved J3 29.1 mm to (190.0, 115.0), turned to 0 degrees
- moved J4 25.7 mm to (177.9, 98.7)
- moved R16 25.7 mm to (196.4, 114.2), turned to 0 degrees
- moved BTN1 22.4 mm to (202.5, 98.2), turned to 180 degrees
- moved R7 21.9 mm to (202.9, 95.4), turned to 180 degrees
- moved R13 21.3 mm to (196.6, 100.8), turned to 0 degrees
- moved U1 20.3 mm to (193.8, 112.7), turned to 90 degrees
- moved C2 19.9 mm to (183.8, 113.6)
- moved D6 19.4 mm to (196.4, 112.8), turned to 180 degrees
- moved JP6 18.7 mm to (196.6, 101.1), turned to 180 degrees
- moved R17 18.3 mm to (196.6, 98.8), turned to 0 degrees
- moved R3 16.0 mm to (196.4, 111.5), turned to 180 degrees
- moved U3 15.7 mm to (190.0, 105.3), turned to 45 degrees
- moved JP7 15.3 mm to (196.6, 98.6), turned to 180 degrees
- moved Y1 15.1 mm to (183.8, 109.6)
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Connections:
- net /I2C ext/SCL renamed /SDA
- net /I2C ext/SDA renamed /SCL
- BTN1 pad 1: /PA11 -> GND
- BTN1 pad 2: unconnected-(BTN1-Pad2) -> /PA11
- J3 pad 2: +3.3V -> unconnected-(J3-Pad2)
- J3 pad 3: /SDA_INT -> VBUS
- J3 pad 4: /SCL_INT -> unconnected-(J3-Pad4)
- U3 pad 27: /RGB -> /PA28
Routing:
- net GND: track 297.4 -> 94.6 mm, vias 53 -> 39
- net /PA15: track 57.4 -> 5.27 mm, vias 4 -> 0
- net VBUS: track 38.3 -> 88.9 mm, vias 2 -> 5
- net /~{RESET}: track 53.0 -> 18.8 mm, vias 3 -> 0
- net /LED Driver/LED_PWR: track 77.9 -> 101.3 mm, vias 2 -> 1
- net /TX: track 0.00 -> 22.9 mm, vias 0 -> 1
- net /PA03: track 0.00 -> 22.2 mm, vias 0 -> 1
- net /PA04: track 0.00 -> 21.5 mm, vias 0 -> 1
- net /PA14: track 27.7 -> 6.78 mm, vias 4 -> 0
- net /PA11: track 45.2 -> 24.6 mm, vias 4 -> 0
- net /RX: track 0.00 -> 20.3 mm, vias 0 -> 1
- net +5V: track 113.2 -> 94.2 mm
- net /D-: track 13.9 -> 30.0 mm
- net /D+: track 15.1 -> 31.0 mm
- net /SWDIO: track 31.4 -> 16.2 mm, vias 2 -> 1
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Other:
- board text added: "02"
- board text added: "DNP"
- board text added: "PA11"
- board text added: "RST"
- board text removed: "11 - 14 - 15"

Commit message: final?
Routing:
- net GND: track 94.6 -> 102.1 mm, vias 39 -> 44
Other:
- board text added: "10uf"
- board text added: "1uf"
- board text added: "3pf"
- board text removed: "Leds Power"
