File: Hardware/LegoLight_R3/LegoLight_R3.kicad_sch (KiCad schematic)
At the start: 22 parts, among them J3 I2C, J4 SWD, J5 C1, J6 I2C_INT, J7 LED_EXT, U1 24LC01BT-I_OT, U3 ATSAMD21E18A-A, Y1 32.768 kHz

Commit message: update pcbs
Parts:
- removed D1: SK6812, LED_SMD:LED_SK6812_PLCC4_5.0x5.0mm_P3.2mm, symbol LED:SK6812
- removed J3: I2C, SnapEDA Library:ADAFRUIT_4328, symbol Connector_Generic:Conn_01x04
- removed J5: C1, Connector_PinHeader_1.27mm:PinHeader_1x03_P1.27mm_Vertical, symbol Connector_Generic:Conn_01x03
- removed J6: I2C_INT, Connector_PinHeader_2.54mm:PinHeader_1x04_P2.54mm_Vertical, symbol Connector_Generic:Conn_01x04
- added C7, C8: 3pf, Capacitor_SMD:C_0805_2012Metric, symbol SparkFun_Qwiic_Micro_SAMD21E-eagle-import:1.0UF-0402-16V-10%
- added J3, J8: 103R012BB100, mouser:103R012BB100, symbol mousser:103R012BB100
- added Y2: 32.768 kHz, Crystal:Crystal_SMD_MicroCrystal_CC8V-T1A-2Pin_2.0x1.2mm, symbol Device:Crystal
- C1, C2: footprint Capacitor_SMD:C_0805_2012Metric_Pad1.18x1.45mm_HandSolder -> Capacitor_SMD:C_0805_2012Metric
- J7: footprint SnapEDA Library:ADAFRUIT_4328 -> SnapEDA Library:SPARKFUN_PRT-14417
- RESET1: footprint SnapEDA Library:SW_TL3305AF160QG -> mouser:B3U-1000P; symbol TL3305AF160QG:TL3305AF160QG -> Switch:SW_Push
- U1: footprint Package_TO_SOT_SMD:SOT-353_SC-70-5_Handsoldering -> Package_TO_SOT_SMD:SOT-353_SC-70-5
- Y1: footprint Crystal:Crystal_SMD_MicroCrystal_CC8V-T1A-2Pin_2.0x1.2mm_HandSoldering -> Crystal:Crystal_SMD_MicroCrystal_CC8V-T1A-2Pin_2.0x1.2mm; Mouser Part Number (none) -> 815-ABS06-32.768K-T
Connections:
- net +3.3V: now also J3.5, J8.3
- net GND: now also RESET1.1, C7.2, C8.2, J3.1, J3.MP1, J3.MP2, J3.MP3, J3.MP4, J8.1, J8.MP1, J8.MP2, J8.MP3, J8.MP4; no longer RESET1.3, RESET1.4
- net PA02: now also J8.11
- net PA03: now also J8.9
- net PA04: now also J8.7
- net PA05: now also J3.7
- net PA06: now also J3.9
- net PA07: now also J3.11
- net PA14: now also C7.1, Y2.2
- net PA15: now also C8.1, Y2.1
- net RX: now also J8.12
- net SCL_INT: now also J8.2
- net SDA_INT: now also J8.4
- net TX: now also J8.10
- net ~{RESET}: no longer RESET1.1
- net I2C ext/SCL_out renamed SCL
- net SCL: now also J8.6
- net I2C ext/SDA_out renamed SDA
- net SDA: now also J8.8
- net RGB renamed PA28
- new net VBUS: J3.3, J8.5
- no-connect marks 3 -> 2

Commit message: final?
Parts:
- RESET1: Mouser Part Number 612-TL3305AF160QG -> 653-B3U-1000P
Changed lines of the file:
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@@
 			)
 		)
-		(property "Mouser Part Number" "612-TL3305AF160QG"
+		(property "Mouser Part Number" "653-B3U-1000P"
 			(at 242.57 34.29 0)
 			(effects
