File: Hardware/LegoLight_R3/buttons.kicad_sch (KiCad schematic)
At the start: 6 parts

Commit message: update pcbs
Parts:
- removed BTN2, BTN3: BTN, SnapEDA Library:SW_TL3305AF160QG, symbol TL3305AF160QG:TL3305AF160QG
- removed R11, R12: 10KOHM, Resistor_SMD:R_0805_2012Metric_Pad1.20x1.40mm_HandSolder, symbol SparkFun_Qwiic_Micro_SAMD21E-eagle-import:10KOHM-0402-1/16W-1%
- BTN1: footprint SnapEDA Library:SW_TL3305AF160QG -> mouser:B3U-1000P; symbol TL3305AF160QG:TL3305AF160QG -> Switch:SW_Push
Connections:
- net BTN_1: now also BTN1.2; no longer BTN1.1
- net GND: now also BTN1.1; no longer BTN1.3, BTN1.4
- no-connect marks 3 -> 0

Commit message: final?
Parts:
- BTN1: Mouser Part Number 612-TL3305AF160QG -> 653-B3U-1000P
Changed lines of the file:
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@@
 			)
 		)
-		(property "Mouser Part Number" "612-TL3305AF160QG"
+		(property "Mouser Part Number" "653-B3U-1000P"
 			(at 45.72 60.96 0)
 			(effects
